File: hardware/main-board/mainboard.sch (EAGLE design)
At the start: 27 parts, among them J2 ADDRESS BUS, J3 DATA BUS, U1 AS6C1008-55PCN, U3 L7805, U4 SST39SF010A-70-4C-NHEMICROCHI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

Commit message: adding clock and power module
Parts:
- removed C1, C2, C3: (no value), passives:C-USC0805K
- removed U$3: SWITCH_TACTILETACTILE-2PIN-NARROW, switches:SWITCH_TACTILETACTILE-2PIN-NARROW
- removed U3: L7805, voltage-regulator:L7805
- added C10, C11, C6, C7, C8, C9: 0.1 uF, passives:C-USC0805K
- added J5: IO_ADDRESS, connector:M16LONGPADS
- added J6: IO_DATA, connector:M08LONGPADS
- added J7: IO_CONTROLS, connector:M08LONGPADS
- added LED1: FLASH MEM, leds:LED1206
- added LED2: SRAM, leds:LED1206
- added LED3, LED4, LED5: (no value), leds:LED1206
- added LED6, LED7: OP Code Fetch, leds:LED1206
- added R10, R14, R15: 1 K, passives:RESISTOR0805-RES
- added R11, R12, R13, R17, R18, R9: 100 R, passives:RESISTOR0805-RES
- added R16: 10 K, passives:RESISTOR0805-RES
- added S2: Program, switches:SWITCH-SPSTKIT
- added S3: WAIT, switches:SWITCH-SPSTKIT
- added U2: CD4001BE, logic:CD4001BE
- J1: device connector:M023.5MM -> connector:M02PTH
- R1: value (none) -> 100 R
- U$2: value QUAD-2-INPUT-NAND-GATESTI-PDIPJ -> SWITCH_TACTILETACTILE-2PIN-NARROW; device logic:QUAD-2-INPUT-NAND-GATESTI-PDIPJ -> switches:SWITCH_TACTILETACTILE-2PIN-NARROW
Connections:
- removed net VIN: C1.1, C3.1, J1.1, U3.IN
- new net BUSAK: IC1.BUSAK, J7.6, R11.1
- new net BUSRQ: IC1.BUSRQ, J7.7, S2.P
- new net FLASH_MEM_CS: R1.2, U$5.B, U2.J=~A+B
- new net FLASH_MEM_CS#: U$5.B_, U4.CE
- new net INT: IC1.INT, J7.2, R15.1
- new net IORQ: U2.H
- new net IRQ_ACK: R18.2, U2.M=~G+H
- new net M1: IC1.M1, U2.F, U2.G
- new net MREQ: IC1.MREQ, U2.A, U2.C, U2.E
- new net N$10: LED3.A, R11.2
- new net N$11: LED4.A, R12.2
- new net N$12: IC1.RFSH, R12.1
- new net N$13: LED2.A, R9.1
- new net N$14: IC1.HALT, R13.1
- new net N$15: LED5.A, R13.2
- new net N$16: R14.1, S3.S
- new net N$17: LED6.A, R17.1
- new net N$18: LED7.A, R18.1
- new net N$20: IC1.IORQ
- new net NMI: C11.1, IC1.NMI, R16.1, U$2.A
- new net OP_CODE_FETCH: R17.2, U2.L=~E+F
- new net READ_ENABLE_LOW: IC1.RD, J7.4, U1.OE, U4.OE
- new net SRAM_CS: R9.2, U$5.C, U2.K=~C+D
- new net SRAM_CS#: U$5.C_, U1.CE
- new net SYS_CLK: IC1.CLK, J7.5
- new net WAIT: IC1.WAIT, J7.3, S3.P
- new net WRITE_ENABLE_LOW: IC1.WR, U1.WE, U4.WE
- net A0: now also J5.1
- net A1: now also J5.2
- net A10: now also J5.11
- net A11: now also J5.12
- net A12: now also J5.13
- net A13: now also J5.14
- net A14-SWITCH: now also J5.15
- net A15-SRAM-A14: now also J5.16
- net A2: now also J5.3
- net A3: now also J5.4
- net A4: now also J5.5
- net A5: now also J5.6
- net A6: now also J5.7
- net A7: now also J5.8
- net A8: now also J5.9
- net A9: now also J5.10
- net D0: now also J6.1
- net D1: now also J6.2
- net D2: now also J6.3
- net D3: now also J6.4
- net D4: now also J6.5
- net D5: now also J6.6
- net D6: now also J6.7
- net D7: now also J6.8
- net GND: now also C10.2, C11.2, C6.2, C7.2, C8.2, C9.2, J7.1, LED1.C, LED2.C, LED3.C, LED4.C, LED5.C, LED6.C, LED7.C, S1.O, S2.O, S3.O, U$2.C, U$4.VSS, U$5.VSS, U2.VSS; no longer C1.2, C2.2, C3.2, U3.GND
- net MEM_SELECT: now also U2.B; no longer U4.CE
- net MEM_SELECT#: now also U2.D; no longer U1.CE
- net N$1: now also LED1.A, R1.1; no longer R1.2
- net N$2: now also R10.1, S2.S; no longer S1.S
- net V5: now also C10.1, C6.1, C7.1, C8.1, C9.1, J1.1, J7.8, R10.2, R14.2, R15.2, R16.2, S1.S, U$4.VCC, U$5.VCC, U2.VDD; no longer C2.1, U$2.AIN1, U3.OUT
Other:
- note added: "IO BOARD needs to pull INT LOW and BUSREQ Low Wait for BUSACK to go low Put address on address lines to read Then pull: READ_ENABLE_LOW"
- note removed: "CLOCK"
- note removed: "Erase EEPROM circuit"
- note removed: "z80VCC | s2on | epromVCC | CE | OE | COMMENT 1 | 1 | 1 | NA | NA | Z80 switch on so all on 1 | 0 | 1 | NA | NA | Z80 switch on so all on 0 | 1 | 1 | NA | NA | Reprogram EEPROM 0 | 0 | 1 | 0 | 12 | Clear EEPROM on WE_ PULSE"

Commit message: closer to layout complete for z80Computer
Parts:
- added LED10, LED11, LED12, LED13, LED14, LED15, LED16, LED17, LED18, LED19, LED20, LED21, LED22, LED23, LED24, LED25, LED26, LED27, LED28, LED29, LED30, LED31, LED8, LED9: (no value), leds:LED1206
- added LED32: Read Enable, leds:LED1206
- added LED33: Output Enable, leds:LED1206
- added R19, R20: 100 R, passives:RESISTOR0805-RES
Connections:
- new net N$19: LED32.A, R19.1
- new net N$21: LED33.A, R20.1
- new net READ_ENABLE_LOW#: R19.2, U$5.F_
- new net WRITE_ENABLE_LOW#: R20.2, U$5.E_
- net A0: now also LED8.A
- net A1: now also LED9.A
- net A10: now also LED18.A
- net A11: now also LED19.A
- net A12: now also LED20.A
- net A13: now also LED21.A
- net A14: now also LED22.A
- net A15: now also LED23.A
- net A2: now also LED10.A
- net A3: now also LED11.A
- net A4: now also LED12.A
- net A5: now also LED13.A
- net A6: now also LED14.A
- net A7: now also LED15.A
- net A8: now also LED16.A
- net A9: now also LED17.A
- net D0: now also LED24.A
- net D1: now also LED25.A
- net D2: now also LED26.A
- net D3: now also LED27.A
- net D4: now also LED28.A
- net D5: now also LED29.A
- net D6: now also LED30.A
- net D7: now also LED31.A
- net GND: now also LED10.C, LED11.C, LED12.C, LED13.C, LED14.C, LED15.C, LED16.C, LED17.C, LED18.C, LED19.C, LED20.C, LED21.C, LED22.C, LED23.C, LED24.C, LED25.C, LED26.C, LED27.C, LED28.C, LED29.C, LED30.C, LED31.C, LED32.C, LED33.C, LED8.C, LED9.C
- net READ_ENABLE_LOW: now also U$5.F
- net WRITE_ENABLE_LOW: now also U$5.E

Commit message: main board starting to route
Connections:
- removed net A14: J2.16, LED22.A
- removed net A15: J2.17, LED23.A
- removed net N$20: IC1.IORQ
- net A14-SWITCH: now also J2.16, LED22.A
- net A15-SRAM-A14: now also J2.17, LED23.A
- net IORQ: now also IC1.IORQ

Commit message: update on clock board, so much cleaner now re-layout of main board
Parts:
- removed J5: IO_ADDRESS, connector:M16LONGPADS
- removed J7: IO_CONTROLS, connector:M08LONGPADS
- removed LED10, LED11, LED12, LED13, LED14, LED15, LED16, LED17, LED18, LED19, LED20, LED21, LED22, LED23, LED24, LED25, LED26, LED27, LED28, LED29, LED3, LED30, LED31, LED4, LED5, LED8, LED9: (no value), leds:LED1206
- removed LED2: SRAM, leds:LED1206
- removed LED32: Read Enable, leds:LED1206
- removed LED33: Output Enable, leds:LED1206
- removed LED6, LED7: OP Code Fetch, leds:LED1206
- removed R11, R12, R13, R17, R18, R19, R20, R9: 100 R, passives:RESISTOR0805-RES
- added C1: 10 uF, passives:C-USC0805K
- J2: value ADDRESS BUS -> (none)
- J3: value DATA BUS -> (none); device connector:M10SILK_FEMALE_PTH -> connector:M08LOCK_LONGPADS
- J6: value IO_DATA -> IO_CONTROLS; device connector:M08LONGPADS -> connector:M12LONGPADS
- LED1: value FLASH MEM -> (none)
- R1: value 100 R -> 1 K
Connections:
- removed net IRQ_ACK: R18.2, U2.M=~G+H
- removed net N$10: LED3.A, R11.2
- removed net N$11: LED4.A, R12.2
- removed net N$12: IC1.RFSH, R12.1
- removed net N$13: LED2.A, R9.1
- removed net N$14: IC1.HALT, R13.1
- removed net N$15: LED5.A, R13.2
- removed net N$17: LED6.A, R17.1
- removed net N$18: LED7.A, R18.1
- removed net N$19: LED32.A, R19.1
- removed net N$21: LED33.A, R20.1
- removed net N$3: C5.1, IC1.VCC, S1.P
- removed net OP_CODE_FETCH: R17.2, U2.L=~E+F
- removed net READ_ENABLE_LOW#: R19.2, U$5.F_
- removed net WRITE_ENABLE_LOW#: R20.2, U$5.E_
- new net HALT: IC1.HALT, J6.11
- new net RFSH: IC1.RFSH, J6.10
- new net VIN: J1.1, S1.S
- net A0: no longer J5.1, LED8.A
- net A1: no longer J5.2, LED9.A
- net A10: no longer J5.11, LED18.A
- net A11: no longer J5.12, LED19.A
- net A12: no longer J5.13, LED20.A
- net A13: no longer J5.14, LED21.A
- net A14-SWITCH: no longer J5.15, LED22.A
- net A15-SRAM-A14: no longer J5.16, LED23.A
- net A2: no longer J5.3, LED10.A
- net A3: no longer J5.4, LED11.A
- net A4: no longer J5.5, LED12.A
- net A5: no longer J5.6, LED13.A
- net A6: no longer J5.7, LED14.A
- net A7: no longer J5.8, LED15.A
- net A8: no longer J5.9, LED16.A
- net A9: no longer J5.10, LED17.A
- net BUSAK: now also J6.6; no longer J7.6, R11.1
- net BUSRQ: now also J6.7; no longer J7.7
- net D0: now also J3.1; no longer J3.2, J6.1, LED24.A
- net D1: now also J3.2; no longer J3.3, J6.2, LED25.A
- net D2: now also J3.3; no longer J3.4, J6.3, LED26.A
- net D3: now also J3.4; no longer J3.5, J6.4, LED27.A
- net D4: now also J3.5; no longer J3.6, J6.5, LED28.A
- net D5: now also J3.6; no longer J3.7, J6.6, LED29.A
- net D6: now also J3.7; no longer J3.8, J6.7, LED30.A
- net D7: now also J3.8; no longer J3.9, J6.8, LED31.A
- net FLASH_MEM_CS: no longer R1.2
- net GND: now also C1.2, J6.1; no longer J3.1, J7.1, LED10.C, LED11.C, LED12.C, LED13.C, LED14.C, LED15.C, LED16.C, LED17.C, LED18.C, LED19.C, LED2.C, LED20.C, LED21.C, LED22.C, LED23.C, LED24.C, LED25.C, LED26.C, LED27.C, LED28.C, LED29.C, LED3.C, LED30.C, LED31.C, LED32.C, LED33.C, LED4.C, LED5.C, LED6.C, LED7.C, LED8.C, LED9.C
- net INT: now also J6.2; no longer J7.2
- net IORQ: now also J6.8; no longer U2.H
- net M1: now also J6.9; no longer U2.F, U2.G
- net MREQ: no longer U2.E
- net READ_ENABLE_LOW: now also J6.4; no longer J7.4, U$5.F
- net SRAM_CS: no longer R9.2
- net SYS_CLK: now also J6.5; no longer J7.5
- net V5: now also C1.1, C5.1, IC1.VCC, J6.12, R1.2, S1.P; no longer J1.1, J3.10, J7.8, S1.S
- net WAIT: now also J6.3; no longer J7.3
- net WRITE_ENABLE_LOW: no longer U$5.E

Commit message: some routing complete
Connections:
- net BUSAK: now also J6.4; no longer J6.6
- net IORQ: now also J6.10; no longer J6.8
- net M1: now also J6.8; no longer J6.9
- net READ_ENABLE_LOW: now also J6.3; no longer J6.4
- net RFSH: now also J6.9; no longer J6.10
- net SRAM-A15: now also J4.9; no longer J4.7
- net SRAM-A16: now also J4.7; no longer J4.9
- net WAIT: now also J6.6; no longer J6.3

Commit message: not sure
Parts:
- added U$3: CMD_C0DE_LOGOCMD_CODE_LOGO_SILK, logos:CMD_C0DE_LOGOCMD_CODE_LOGO_SILK
- J2: value (none) -> IO_ADDRESS
- J3: value (none) -> IO_DATA
- LED1: value (none) -> pwr
- S1: value (none) -> MAIN PWR
Connections:
- net GND: now also J2.18; no longer J2.1
- net V5: now also J2.1; no longer J2.18
Changed lines of the file:
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@@
 <parts>
 <part name="IC1" library="zilog" library_urn="urn:adsk.eagle:library:419" deviceset="Z80CPU" device="" package3d_urn="urn:adsk.eagle:package:19651/1"/>
-<part name="S1" library="switches" deviceset="SWITCH-SPST" device="KIT"/>
+<part name="S1" library="switches" deviceset="SWITCH-SPST" device="KIT" value="MAIN PWR"/>
 <part name="U$4" library="logic" deviceset="QUAD-2-INPUT-OR-GATES" device="TI-R-PDIPT14" package3d_urn="urn:adsk.eagle:package:16498247/1"/>
 <part name="U$5" library="logic" deviceset="HEX-INVERTER" device="TI-J0014A" package3d_urn="urn:adsk.eagle:package:16498301/1"/>
@@
 <part name="C11" library="passives" deviceset="C-US" device="C0805K" package3d_urn="urn:adsk.eagle:package:8089589/1" value="0.1 uF"/>
 <part name="J1" library="connector" deviceset="M02" device="PTH"/>
-<part name="J2" library="connector" deviceset="M18" device="_"/>
-<part name="J3" library="connector" deviceset="M08" device="LOCK_LONGPADS"/>
-<part name="LED1" library="leds" deviceset="LED" device="1206"/>
+<part name="J2" library="connector" deviceset="M18" device="_" value="IO_ADDRESS"/>
+<part name="J3" library="connector" deviceset="M08" device="LOCK_LONGPADS" value="IO_DATA"/>
+<part name="LED1" library="leds" deviceset="LED" device="1206" value="pwr"/>
 <part name="R1" library="passives" deviceset="RESISTOR" device="0805-RES" value="1 K"/>
 <part name="C1" library="passives" deviceset="C-US" device="C0805K" package3d_urn="urn:adsk.eagle:package:8089589/1" value="10 uF"/>
 <part name="J6" library="connector" deviceset="M12" device="LONGPADS" value="IO_CONTROLS"/>
+<part name="U$3" library="logos" deviceset="CMD_C0DE_LOGO" device="CMD_CODE_LOGO_SILK"/>
 </parts>
 <sheets>
@@
 </segment>
 <segment>
-<wire x1="205.74" y1="-60.96" x2="205.74" y2="-58.42" width="0.1524" layer="91"/>
-<label x="205.74" y="-53.34" size="1.778" layer="95" rot="R90"/>
-<pinref part="J2" gate="G$1" pin="1"/>
+<wire x1="162.56" y1="-60.96" x2="162.56" y2="-58.42" width="0.1524" layer="91"/>
+<label x="162.56" y="-53.34" size="1.778" layer="95" rot="R90"/>
+<pinref part="J2" gate="G$1" pin="18"/>
 </segment>
 </net>
@@
 <wire x1="78.74" y1="-2.54" x2="78.74" y2="2.54" width="0.1524" layer="91"/>
 <label x="78.74" y="2.54" size="1.778" layer="95"/>
-</segment>
-<segment>
-<wire x1="162.56" y1="-60.96" x2="162.56" y2="-58.42" width="0.1524" layer="91"/>
-<label x="162.56" y="-53.34" size="1.778" layer="95" rot="R90"/>
-<pinref part="J2" gate="G$1" pin="18"/>
 </segment>
 <segment>
@@
 <label x="20.32" y="20.32" size="1.778" layer="95"/>
 </segment>
+<segment>
+<wire x1="205.74" y1="-60.96" x2="205.74" y2="-58.42" width="0.1524" layer="91"/>
+<label x="205.74" y="-53.34" size="1.778" layer="95" rot="R90"/>
+<pinref part="J2" gate="G$1" pin="1"/>
+</segment>
 </net>
 <net name="D0" class="0">
@@
 </nets>
 </sheet>
+<sheet>
+<plain>
+</plain>
+<instances>
+<instance part="U$3" gate="G$1" x="27.94" y="50.8" smashed="yes"/>
+</instances>
+<busses>
+</busses>
+<nets>
+</nets>
+</sheet>
